Commit message: working bycicle drive

File: src/uno/urdf/diff_drive_robot.urdf (robot description, URDF)
Before this commit: robot diff_drive_robot, 6 links, 5 joints
Links:
- removed link chassis-link
- removed link front-left-wheel-link
- removed link front-right-wheel-link
- removed link rear-left-wheel-link
- removed link rear-right-wheel-link
- added link chassis_link, mass 0.4; collision box size=0.2 0.12 0.01; visual box size=0.2 0.12 0.01
- added link front_left_wheel_link, mass 0.2; collision cylinder length=0.01 radius=0.03; visual cylinder length=0.01 radius=0.03
- added link front_right_wheel_link, mass 0.2; collision cylinder length=0.01 radius=0.03; visual cylinder length=0.01 radius=0.03
- added link rear_left_wheel_link, mass 0.2; collision cylinder length=0.01 radius=0.03; visual cylinder length=0.01 radius=0.03
- added link rear_right_wheel_link, mass 0.2; collision cylinder length=0.01 radius=0.03; visual cylinder length=0.01 radius=0.03
- added link virtual_front_wheel, mass 0.2; visual cylinder length=0.01 radius=0.03
- added link virtual_rear_wheel, mass 0.2; visual cylinder length=0.01 radius=0.03
Joints:
- removed joint joint-base-chassis
- removed joint joint-chassis-front-left-wheel
- removed joint joint-chassis-front-right-wheel
- removed joint joint-chassis-rear-left-wheel
- removed joint joint-chassis-rear-right-wheel
- added joint joint_base_chassis: type fixed, parent base_link, child chassis_link, origin xyz=0 0 0.03 rpy=0 0 0
- added joint joint_chassis_front_left_wheel: type continuous, parent chassis_link, child front_left_wheel_link, origin xyz=0.06 -0.065 0 rpy=0 0 0, axis 0 1 0
- added joint joint_chassis_front_right_wheel: type continuous, parent chassis_link, child front_right_wheel_link, origin xyz=0.06 0.065 0 rpy=0 0 0, axis 0 1 0
- added joint joint_chassis_rear_left_wheel: type continuous, parent chassis_link, child rear_left_wheel_link, origin xyz=-0.06 -0.065 0 rpy=0 0 0, axis 0 1 0
- added joint joint_chassis_rear_right_wheel: type continuous, parent chassis_link, child rear_right_wheel_link, origin xyz=-0.06 0.065 0 rpy=0 0 0, axis 0 1 0
- added joint virtual_front_wheel_joint: type revolute, parent chassis_link, child virtual_front_wheel, origin xyz=0.3 0 -0.15, axis 0 0 1, limit lower=-0.4 upper=0.4 effort=100.0 velocity=0.0
- added joint virtual_rear_wheel_joint: type continuous, parent chassis_link, child virtual_rear_wheel, origin xyz=-0.06 0 0 rpy=0 0 1.5708, axis 1 0 0, limit effort=100.0 velocity=100.0

Commit message: committing changes for depth cam and imu sensor

File: src/uno/urdf/diff_drive_robot.urdf (robot description, URDF)
Before this commit: robot diff_drive_robot, 8 links, 7 joints
Links:
- added link camera_link_optical
- added link imu_link
Joints:
- added joint camera_optical_joint: type fixed, parent chassis_link, child camera_link_optical, origin xyz=0 0 0 rpy=-1.571 0 -1.571
- added joint imu_joint: type fixed, parent chassis_link, child imu_link, origin xyz=0 0 1.2 rpy=0 0 0

Commit message: adding touch sensor to wall

File: src/uno/urdf/diff_drive_robot.urdf (robot description, URDF)
Before this commit: robot diff_drive_robot, 10 links, 9 joints
Links:
- added link world
Joints:
- added joint base_joint: type fixed, parent world, child base_link, origin xyz=1.5 1.0 0 rpy=0 0 0

Commit message: adding touch sensor to wall

File: src/uno/urdf/diff_drive_robot.urdf (robot description, URDF)
Before this commit: robot diff_drive_robot, 11 links, 10 joints
Joints:
- joint joint_base_chassis: origin xyz=0 0 0.03 rpy=0 0 0 -> xyz=0 0 0 rpy=0 0 0

Commit message: adding touch sensor to wall

File: src/uno/urdf/diff_drive_robot.urdf (robot description, URDF)
Before this commit: robot diff_drive_robot, 11 links, 10 joints
Links:
- link base_link: mass None -> 0.4; geometry collision box size=0.2 0.12 0.01; visual box size=0.2 0.12 0.01

Commit message: adding touch sensor to wall

File: src/uno/urdf/diff_drive_robot.urdf (robot description, URDF)
Before this commit: robot diff_drive_robot, 11 links, 10 joints
Links:
- removed link virtual_front_wheel
- removed link virtual_rear_wheel
- link base_link: mass 0.4 -> 0.6; geometry collision box size=0.25 0.15 0.02; visual box size=0.25 0.15 0.02
- link chassis_link: mass 0.4 -> 0.6; geometry collision box size=0.25 0.15 0.02; visual box size=0.25 0.15 0.02
- link front_left_wheel_link: mass 0.2 -> 0.3; geometry collision cylinder length=0.02 radius=0.04; visual cylinder length=0.02 radius=0.04
- link front_right_wheel_link: mass 0.2 -> 0.3; geometry collision cylinder length=0.02 radius=0.04; visual cylinder length=0.02 radius=0.04
- link rear_left_wheel_link: mass 0.2 -> 0.3; geometry collision cylinder length=0.02 radius=0.04; visual cylinder length=0.02 radius=0.04
- link rear_right_wheel_link: mass 0.2 -> 0.3; geometry collision cylinder length=0.02 radius=0.04; visual cylinder length=0.02 radius=0.04
Joints:
- removed joint base_joint
- removed joint camera_optical_joint
- removed joint imu_joint
- removed joint joint_base_chassis
- removed joint virtual_front_wheel_joint
- removed joint virtual_rear_wheel_joint
- joint joint_chassis_front_left_wheel: limit (none) -> effort=50.0 velocity=3.0
- joint joint_chassis_front_right_wheel: limit (none) -> effort=50.0 velocity=3.0
- joint joint_chassis_rear_left_wheel: limit (none) -> effort=50.0 velocity=3.0
- joint joint_chassis_rear_right_wheel: limit (none) -> effort=50.0 velocity=3.0

Commit message: adding touch sensor to wall

File: src/uno/urdf/diff_drive_robot.urdf (robot description, URDF)
Before this commit: robot diff_drive_robot, 9 links, 4 joints
Links:
- added link virtual_front_wheel, mass 0.2; visual cylinder length=0.01 radius=0.03
- added link virtual_rear_wheel, mass 0.2; visual cylinder length=0.01 radius=0.03
- link base_link: mass 0.6 -> 0.4; geometry collision box size=0.2 0.12 0.01; visual box size=0.2 0.12 0.01
- link chassis_link: mass 0.6 -> 0.4; geometry collision box size=0.2 0.12 0.01; visual box size=0.2 0.12 0.01
- link front_left_wheel_link: mass 0.3 -> 0.2; geometry collision cylinder length=0.01 radius=0.03; visual cylinder length=0.01 radius=0.03
- link front_right_wheel_link: mass 0.3 -> 0.2; geometry collision cylinder length=0.01 radius=0.03; visual cylinder length=0.01 radius=0.03
- link rear_left_wheel_link: mass 0.3 -> 0.2; geometry collision cylinder length=0.01 radius=0.03; visual cylinder length=0.01 radius=0.03
- link rear_right_wheel_link: mass 0.3 -> 0.2; geometry collision cylinder length=0.01 radius=0.03; visual cylinder length=0.01 radius=0.03
Joints:
- added joint base_joint: type fixed, parent world, child base_link, origin xyz=1.5 1.0 0 rpy=0 0 0
- added joint camera_optical_joint: type fixed, parent chassis_link, child camera_link_optical, origin xyz=0 0 0 rpy=-1.571 0 -1.571
- added joint imu_joint: type fixed, parent chassis_link, child imu_link, origin xyz=0 0 1.2 rpy=0 0 0
- added joint joint_base_chassis: type fixed, parent base_link, child chassis_link, origin xyz=0 0 0 rpy=0 0 0
- added joint virtual_front_wheel_joint: type revolute, parent chassis_link, child virtual_front_wheel, origin xyz=0.3 0 -0.15, axis 0 0 1, limit lower=-0.4 upper=0.4 effort=100.0 velocity=0.0
- added joint virtual_rear_wheel_joint: type continuous, parent chassis_link, child virtual_rear_wheel, origin xyz=-0.06 0 0 rpy=0 0 1.5708, axis 1 0 0, limit effort=100.0 velocity=100.0
- joint joint_chassis_front_left_wheel: limit effort=50.0 velocity=3.0 -> (none)
- joint joint_chassis_front_right_wheel: limit effort=50.0 velocity=3.0 -> (none)
- joint joint_chassis_rear_left_wheel: limit effort=50.0 velocity=3.0 -> (none)
- joint joint_chassis_rear_right_wheel: limit effort=50.0 velocity=3.0 -> (none)

Commit message: adding touch sensor to wall

File: src/uno/urdf/diff_drive_robot.urdf (robot description, URDF)
Before this commit: robot diff_drive_robot, 11 links, 10 joints
Links:
- link virtual_front_wheel: geometry collision cylinder length=0.01 radius=0.03; visual cylinder length=0.01 radius=0.03
- link virtual_rear_wheel: geometry collision cylinder length=0.01 radius=0.03; visual cylinder length=0.01 radius=0.03
Joints:
- joint virtual_front_wheel_joint: origin xyz=0.3 0 -0.15 -> xyz=-0.06 0 0 rpy=0 0 1.5708

Commit message: adding touch sensor to wall

File: src/uno/urdf/diff_drive_robot.urdf (robot description, URDF)
Before this commit: robot diff_drive_robot, 11 links, 10 joints
Links:
- link base_link: mass 0.4 -> None; geometry 

Commit message: adding touch sensor to wall

File: src/uno/urdf/diff_drive_robot.urdf (robot description, URDF)
Before this commit: robot diff_drive_robot, 10 links, 9 joints
Joints:
- joint joint_base_chassis: origin xyz=0 0 0 rpy=0 0 0 -> xyz=0.06 0.065 0 rpy=0 0 0

Commit message: adding touch sensor to wall

File: src/uno/urdf/diff_drive_robot.urdf (robot description, URDF)
Before this commit: robot diff_drive_robot, 10 links, 9 joints
Links:
- removed link base_link
- added link map
Joints:
- joint joint_base_chassis: parent base_link -> map

Commit message: gazeebo fix

File: src/uno/urdf/diff_drive_robot.urdf (robot description, URDF)
Before this commit: robot diff_drive_robot, 10 links, 9 joints
Links:
- added link camera_link, mass 0.2; collision cylinder length=0.01 radius=0.003; visual cylinder length=0.01 radius=0.003
Joints:
- added joint joint_chassis_camera: type continuous, parent chassis_link, child camera_link, origin xyz=0.06 0.065 0 rpy=0 0 0, axis 0 1 0

Commit message: adding fix for imu

File: src/uno/urdf/diff_drive_robot.urdf (robot description, URDF)
Before this commit: robot diff_drive_robot, 11 links, 10 joints
Links:
- link imu_link: mass None -> 0.4
Joints:
- removed joint imu_joint
- added joint joint_chassis_imu: type continuous, parent chassis_link, child imu_link, origin xyz=0.06 0.065 0 rpy=0 0 0, axis 0 1 0

Commit message: segmentation camera

File: src/uno/urdf/diff_drive_robot.urdf (robot description, URDF)
Before this commit: robot diff_drive_robot, 11 links, 10 joints
Links:
- added link instance_segmentation_camera_link, mass 0.2; collision cylinder length=0.01 radius=0.003; visual cylinder length=0.01 radius=0.003
- added link instance_segmentation_camera_link_optical
Joints:
- added joint chasis_instance_camera_joint: type continuous, parent chassis_link, child instance_segmentation_camera_link, origin xyz=0.06 0.065 0 rpy=0 0 0, axis 0 1 0
- added joint instance_camera_optical_joint: type fixed, parent chassis_link, child instance_segmentation_camera_link_optical, origin xyz=0 0 0 rpy=-1.571 0 -1.571

Commit message: segmentation camera

File: src/uno/urdf/diff_drive_robot.urdf (robot description, URDF)
Before this commit: robot diff_drive_robot, 13 links, 12 joints
Links:
- removed link instance_segmentation_camera_link
- removed link instance_segmentation_camera_link_optical
Joints:
- removed joint chasis_instance_camera_joint
- removed joint instance_camera_optical_joint
