Commit message: fix nav2

File: src/uno/urdf/roberto.urdf (robot description, URDF)
Before this commit: robot diff_drive_robot, 9 links, 8 joints
Links:
- removed link map
- added link base_footprint
- added link base_laser_link, mass 0.000001; visual box size=0.00 0.05 0.06
- added link base_link
Joints:
- added joint base_footprint_joint: type fixed, parent base_footprint, child base_link, origin xyz=0 0 0 rpy=0 0 0
- added joint laser: type fixed, parent chassis_link, child base_laser_link, origin xyz=-0.005 0.00 0.360 rpy=3.14159 0 0
- joint joint_base_chassis: parent map -> base_link

Commit message: nav2 integration

File: src/uno/urdf/roberto.urdf (robot description, URDF)
Before this commit: robot diff_drive_robot, 11 links, 10 joints
Links:
- removed link base_laser_link
- removed link camera_link_optical
- added link laser_link, mass 0.000001; visual box size=0.00 0.05 0.06
- added link optical_link
Joints:
- joint camera_optical_joint: child camera_link_optical -> optical_link; parent chassis_link -> base_link
- joint joint_chassis_camera: parent chassis_link -> optical_link
- joint joint_chassis_imu: parent chassis_link -> base_link
- joint laser: child base_laser_link -> laser_link; parent chassis_link -> optical_link

Commit message: removing nav2

File: src/uno/urdf/roberto.urdf (robot description, URDF)
Before this commit: robot diff_drive_robot, 11 links, 10 joints
Joints:
- joint camera_optical_joint: origin xyz=0 0 0 rpy=-1.571 0 -1.571 -> xyz=0.22 0 0 rpy=0 0 0; parent base_link -> chassis_link
- joint joint_chassis_camera: origin xyz=0.3 0 0.1 rpy=0 0 0 -> xyz=0.05 0 0.1 rpy=0 0 0
- joint joint_chassis_imu: parent base_link -> chassis_link
- joint laser: origin xyz=-0.005 0.00 0.360 rpy=3.14159 0 0 -> xyz=0.05 0 0.0360 rpy=3.14159 0 0
